File: KiCad/CoffeeRoasterV2.kicad_sch (KiCad schematic)
At the start: 6 parts, among them J1 Ribbon Cable, J2 Pot center wipers, J3 Pot outer pins, J4 Small Display, J5 Manual LED, J6 Computer LED

Commit message: Updated hardware documentation
Parts:
- added R2, R3: 300, symbol Device:R_US
Connections:
- net at J5.1 (Pin_1): now also R3.1; no longer J1.8 (Pin_8)
- net at J1.10 (Pin_10): now also R2.2; no longer J6.1 (Pin_1)
- new net: J1.8 (Pin_8), R3.2
- new net: J6.1 (Pin_1), R2.1
Changed lines of the file:
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@@
+    (stroke (width 0) (type default))
+  )
+  (wire (pts (xy 176.53 86.36) (xy 176.53 71.12))
     (stroke (width 0) (type default))
   )
@@
     (stroke (width 0) (type default))
   )
-  (wire (pts (xy 179.07 72.39) (xy 123.19 72.39))
+  (wire (pts (xy 123.19 72.39) (xy 179.07 72.39))
     (stroke (width 0) (type default))
   )
@@
     (stroke (width 0) (type default))
   )
-  (wire (pts (xy 176.53 95.25) (xy 176.53 71.12))
+  (wire (pts (xy 176.53 95.25) (xy 176.53 93.98))
     (stroke (width 0) (type default))
   )
@@
     (stroke (width 0) (type default))
   )
-  (wire (pts (xy 176.53 71.12) (xy 139.7 71.12))
-    (stroke (width 0) (type default))
-  )
   (wire (pts (xy 143.51 82.55) (xy 149.86 82.55))
     (stroke (width 0) (type default))
@@
     (stroke (width 0) (type default))
   )
-  (wire (pts (xy 179.07 97.79) (xy 179.07 72.39))
+  (wire (pts (xy 179.07 97.79) (xy 179.07 87.63))
     (stroke (width 0) (type default))
   )
@@
     (stroke (width 0) (type default))
   )
+  (wire (pts (xy 139.7 66.04) (xy 139.7 71.12))
+    (stroke (width 0) (type default))
+  )
   (wire (pts (xy 142.24 80.01) (xy 135.89 80.01))
     (stroke (width 0) (type default))
   )
+  (wire (pts (xy 139.7 71.12) (xy 176.53 71.12))
+    (stroke (width 0) (type default))
+  )
   (wire (pts (xy 142.24 85.09) (xy 129.54 85.09))
     (stroke (width 0) (type default))
@@
     (stroke (width 0) (type default))
   )
+  (wire (pts (xy 179.07 80.01) (xy 179.07 72.39))
+    (stroke (width 0) (type default))
+  )
   (wire (pts (xy 167.64 95.25) (xy 176.53 95.25))
     (stroke (width 0) (type default))
@@
   )
   (wire (pts (xy 167.64 97.79) (xy 179.07 97.79))
-    (stroke (width 0) (type default))
-  )
-  (wire (pts (xy 139.7 71.12) (xy 139.7 66.04))
     (stroke (width 0) (type default))
   )
@@
     )
   )
+  (symbol (lib_id "Device:R_US") (at 179.07 83.82 0) (unit 1)
+    (in_bom yes) (on_board yes) (dnp no) (fields_autoplaced)
+    (property "Reference" "R2" (at 181.61 83.185 0)
+      (effects (font (size 1.27 1.27)) (justify left))
+    )
+    (property "Value" "300" (at 181.61 85.725 0)
+      (effects (font (size 1.27 1.27)) (justify left))
+    )
+    (property "Footprint" "" (at 180.086 84.074 90)
+      (effects (font (size 1.27 1.27)) hide)
+    )
+    (property "Datasheet" "~" (at 179.07 83.82 0)
+      (effects (font (size 1.27 1.27)) hide)
+    )
+    (pin "1")
+    (pin "2")
+    (instances
+      (project "CoffeeRoasterV2"
+        (path "/8f666fca-ffac-4b7f-9a27-dbb30ff4c8fa"
+          (reference "R2") (unit 1)
+        )
+      )
+    )
+  )
   (symbol (lib_id "Connector:Conn_01x02_Pin") (at 147.32 66.04 0) (unit 1)
     (in_bom yes) (on_board yes) (dnp no)
@@
         )
       )
+    )
+  )
+  (symbol (lib_id "Device:R_US") (at 176.53 90.17 0) (unit 1)
+    (in_bom yes) (on_board yes) (dnp no) (fields_autoplaced)
+    (property "Reference" "R3" (at 179.07 89.535 0)
+      (effects (font (size 1.27 1.27)) (justify left))
+    )
+    (property "Value" "300" (at 179.07 92.075 0)
+      (effects (font (size 1.27 1.27)) (justify left))
+    )
+    (property "Footprint" "" (at 177.546 90.424 90)
+      (effects (font (size 1.27 1.27)) hide)
+    )
+    (property "Datasheet" "~" (at 176.53 90.17 0)
+      (effects (font (size 1.27 1.27)) hide)
+    )
+    (pin "1")
+    (pin "2")
+    (instances
+      (project "CoffeeRoasterV2"
+        (path "/8f666fca-ffac-4b7f-9a27-dbb30ff4c8fa"
+          (reference "R3") (unit 1)
+        )
+      )

Commit message: Circuit correction
Corrected LED resistor values on front panel interface board.
Parts:
- R2, R3: value 300 -> 220
Changed lines of the file:
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@@
       (effects (font (size 1.27 1.27)) (justify left))
     )
-    (property "Value" "300" (at 181.61 85.725 0)
+    (property "Value" "220" (at 181.61 85.725 0)
       (effects (font (size 1.27 1.27)) (justify left))
     )
@@
       (effects (font (size 1.27 1.27)) (justify left))
     )
-    (property "Value" "300" (at 179.07 92.075 0)
+    (property "Value" "220" (at 179.07 92.075 0)
       (effects (font (size 1.27 1.27)) (justify left))
     )
